File: CAD/SENSOR_MoonTempTracer/SENSOR_MoonTempTracer.kicad_sch (KiCad schematic)
At the start: 0 parts

Commit message: Rev F: Millstone-Differential Bridge (BBDSD) — digital zeroing, split power domains
Renames the circuit to Millstone-Differential Bridge, tagline "A Balanced
Bridge Dimensionless Signal Detector" (BBDSD). Removes the physical POT1/R7
null-trim in favor of digital zero-offset (same MQTT/flash mechanism as
moon_temp_ads1115). Splits power domains: ADS1115 moves to the always-on
+3V3 rail so it's never power-cycled, while the MOSFET now gates only the
bridge excitation path (SWITCHED_VEXC) — isolates read-timing accuracy to
just the bridge's own RC settling, no ADC startup uncertainty.

Also includes KiCad project files populated by opening in KiCad (10.0.5),
the ERC report, and a new web summary page with an appendix/footnote system
linking back to the original Rev D design.

Co-Authored-By: Claude Sonnet 5 <noreply@anthropic.com>
Claude-Session: https://claude.ai/code/session_01BbEX6hxNqq8y29X9R6AS4t
Parts:
- added C1: 10uF ceramic X7R, CAP_GRM155R60J106ME05D_MUR, symbol GRM155R60J106ME05D
- added C2: 100nF ceramic X7R, symbol GenericC
- added Q1: P-MOSFET e.g. DMG2305UX, symbol PMOS_PLACEHOLDER
- added R1: Rf_A 10.0k 0.01% +-5ppm, STA_RNCF0603_STP, symbol RNCF0603TKY10K0
- added R2: Rf_B 10.0k 0.01% +-5ppm, STA_RNCF0603_STP, symbol RNCF0603TKY10K0
- added R3: 1.2k (LM4040 bias), symbol GenericR
- added R4: 4.7k SDA pullup, symbol GenericR
- added R5: 4.7k SCL pullup, symbol GenericR
- added R6: 10k Q1 gate pullup, symbol GenericR
- added RT1: RT_A moonlit, B57861S0103F045, symbol NTC_PLACEHOLDER
- added RT2: RT_B shaded, B57861S0103F045, symbol NTC_PLACEHOLDER
- added U1: ADS1115IDGSR (I2C 0x48), DGS0010A_N, symbol ADS1115IDGSR
- added U2: LM4040AEM3-2.048 A-grade, symbol LM4040_PLACEHOLDER
Connections:
- new net +3V3: Q1.1 (S), R4.1, R5.1, R6.1, U1.8 (VDD)
- new net GND: C1.2, C2.2, RT1.2, RT2.2, U1.3 (GND), U2.2 (A (anode / GND))
- new net GND (ADDR->GND = addr 0x48): U1.1 (ADDR)
- new net GPIO_PWR_EN: Q1.3 (G), R6.2
- new net SCL: R5.2, U1.10 (SCL)
- new net SDA: R4.2, U1.9 (SDA)
- new net SWITCHED_VEXC: Q1.2 (D), R3.1
- new net VEXC: C1.1, C2.1, R1.1, R2.1, R3.2, U2.1 (K (cathode / Vexc))
- new net mid_A: R1.2, RT1.1, U1.4 (AIN0), U1.5 (AIN1)
- new net mid_B: R2.2, RT2.1, U1.6 (AIN2), U1.7 (AIN3)
- no-connect marks 0 -> 1
Other:
- note added: "+3V3 = always-on (feeds ESP32 AND U1/ADS1115 -- ADC never power-cycled, Rev F)."
- note added: "ADS1115IDGSR"
- note added: "AIN0=abs T_A"
- note added: "AIN1=diff AINP"
- note added: "AIN2=abs T_B"
- note added: "AIN3=diff AINN"
- note added: "ALERT/RDY - NC (unused, polled single-shot)"
- note added: "BRIDGE NETWORK (central board)"
- note added: "EXCITATION REFERENCE"
- note added: "Null-trim (POT1/R7) removed -- zeroing is done digitally via MQTT-settable"
- note added: "PLACEHOLDER SYMBOLS: LM4040, both thermistors, Q1, and R3/R4/R5/R6 are generic boxes with correct pin count/values -- swap for real parts before layout. ADS1115, Rf_A, Rf_B, C1 use exact library symbols."
- note added: "POWER GATE + I2C PULLUPS"
- note added: "PWR_FLAG marks a net as legitimately externally-powered for ERC -- standard KiCad convention"
- note added: "REMOTE THERMISTORS -- ~12in flying leads, matching net labels represent the cable, not a drawn wire"
- note added: "SDA/SCL -> to ESP32-C3 host (existing GPIO21/GPIO20)"
- note added: "SWITCHED_VEXC = gated by Q1, feeds ONLY the bridge excitation (R4/LM4040/Vexc)."
- note added: "U1.VDD on always-on +3V3 -- ADC never power-cycled (Rev F)"
- note added: "ZEROING -- digital offset, not hardware trim (Rev F) -- see notes below"
- note added: "offset persisted to flash, same mechanism as moon_temp_ads1115 (Rev F)."
